File: ruler3.brd (EAGLE design)
At the start: 304.8 x 38.1 mm, 12 parts

Commit message: Added Fractions and line widths
Added common fractions and their decimal counterparts as well as adding line widths to the side.  Fixed the morse code error (M was wrong), increased protractor cutout to 2mm.
Parts:
- moved U$7 34.3 mm to (139.7, 24.1)
- moved U$6 30.6 mm to (152.4, 26.7)
- moved U$3 29.2 mm to (165.1, 24.1)
- moved U$8 10.2 mm to (257.8, 19.1)
- moved U$1 7.62 mm to (204.5, 16.5)
- moved U$4 7.62 mm to (218.4, 16.5)
- moved U$5 7.62 mm to (190.5, 16.5)
- moved U$2 5.08 mm to (177.8, 16.5)
Other:
- board text added: "... .._. ."
- board text added: "0.005"
- board text added: "0.01"
- board text added: "0.02"
- board text added: "0.03"
- board text added: "0.04"
- board text added: "0.05"
- board text added: "0.1"
- board text added: "0.2"
- board text added: "0.3"
- board text added: "0.4"
- board text added: "0.5"
- board text added: "1.0"
- board text added: "1/3 = 0.333* 1/4 = 0.25 1/6 = 0.166* 1/8 = 0.125 1/9 = 0.111* 1/12 = 0.0833* 1/16 = 0.0625 1/24 = 0.04166* 1/32 = 0.03125 1/64 = 0.015625"
- board text added: "1mil = 0.0254mm"
- board text added: "1mil = 1/1000 in"
- board text added: "1mm = 39.3701mil"
- board text added: "2.0"
- board text added: "2/3 = 0.666* 3/8 = 0.375 5/8 = 0.625 7/8 = 0.875 3/16 = 0.1875 5/16 = 0.3125 3/32 = 0.09375 5/32 = 0.15625 3/64 = 0.046875 5/64 = 0.078125"
- board text added: "Inches"
- board text added: "Metric"
- board text added: "R(series)=R1+R2+...Rn R(parallell)= 1/(1/R1+1/R2+...1/Rn)"
- board text added: "Temperature: F-32=C*1.8"
- board text added: "V=IR P=IV"
- board text removed: "--..."
- board text removed: "V=IR P=IV R(series)=R1+R2+...Rn R(parallell)= 1/(1/R1+1/R2+...1/Rn)"
- board text removed: "g=9.8m/s^2 = 32.27 ft/s^2 Temperature: F-32=C*1.8"

Commit message: Checklist
Update dimensions and a few text sizes to comply with the checklist
Parts:
- added U$10, U$11: (no value), SparkFun-Aesthetics:SFE_LOGO_FLAME_.2
- added U$9: (no value), SparkFun-Aesthetics:SFE_LOGO_NAME_.2
- moved FRAME1 167.6 mm to (114.3, -8.89), flipped to the top
Other:
- board text added: "Michelle Shorter"
- board text added: "V01"
Changed lines of the file:
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@@
 <setting verticaltext="up"/>
 </settings>
-<grid distance="10" unitdist="mil" unit="inch" style="lines" multiple="1" display="yes" altdistance="0.005" altunitdist="inch" altunit="inch"/>
+<grid distance="0.1" unitdist="inch" unit="inch" style="lines" multiple="1" display="yes" altdistance="0.1" altunitdist="mm" altunit="mm"/>
 <layers>
-<layer number="1" name="Top" color="4" fill="1" visible="no" active="yes"/>
+<layer number="1" name="Top" color="4" fill="1" visible="yes" active="yes"/>
 <layer number="16" name="Bottom" color="1" fill="1" visible="yes" active="yes"/>
 <layer number="17" name="Pads" color="2" fill="1" visible="yes" active="yes"/>
@@
 <layer number="19" name="Unrouted" color="6" fill="1" visible="yes" active="yes"/>
 <layer number="20" name="Dimension" color="15" fill="1" visible="yes" active="yes"/>
-<layer number="21" name="tPlace" color="16" fill="1" visible="no" active="yes"/>
-<layer number="22" name="bPlace" color="5" fill="1" visible="yes" active="yes"/>
+<layer number="21" name="tPlace" color="16" fill="1" visible="yes" active="yes"/>
+<layer number="22" name="bPlace" color="14" fill="1" visible="yes" active="yes"/>
 <layer number="23" name="tOrigins" color="15" fill="1" visible="yes" active="yes"/>
 <layer number="24" name="bOrigins" color="15" fill="1" visible="yes" active="yes"/>
@@
 <board>
 <plain>
-<wire x1="304.8" y1="0" x2="0" y2="0" width="0.254" layer="20"/>
-<wire x1="0" y1="0" x2="0" y2="38.1" width="0.254" layer="20"/>
-<wire x1="0" y1="38.1" x2="304.8" y2="38.1" width="0.254" layer="20"/>
-<wire x1="304.8" y1="38.1" x2="304.8" y2="0" width="0.254" layer="20"/>
+<wire x1="304.8" y1="0" x2="0" y2="0" width="0.2032" layer="20"/>
+<wire x1="0" y1="0" x2="0" y2="38.1" width="0.2032" layer="20"/>
+<wire x1="0" y1="38.1" x2="304.8" y2="38.1" width="0.2032" layer="20"/>
+<wire x1="304.8" y1="38.1" x2="304.8" y2="0" width="0.2032" layer="20"/>
 <text x="303.276" y="5.08" size="1.27" layer="22" font="vector" ratio="15" rot="MR0">4-40</text>
 <text x="4.826" y="4.826" size="1.27" layer="22" font="vector" ratio="15" rot="MR0">4-40</text>
@@
 </polygon>
 <text x="207.01" y="27.94" size="3.81" layer="21" font="vector" ratio="20" align="bottom-center">One Ruler to Rule Them All</text>
-<text x="292.894" y="7.763" size="1.778" layer="21" font="vector" ratio="15" align="center">Resistance is
+<text x="292.894" y="6.763" size="1.778" layer="21" font="vector" ratio="15" align="center">Resistance is
 not Futile! It
 is voltage
@@
 <rectangle x1="299.8" y1="22.1" x2="304.9" y2="23.1" layer="21"/>
 <rectangle x1="299.8" y1="19.1" x2="304.9" y2="21.1" layer="21"/>
-<text x="303.7" y="17.3" size="1.27" layer="21" font="vector" align="bottom-right">1mm = 39.3701mil</text>
-<text x="303.7" y="14.7" size="1.27" layer="21" font="vector" align="bottom-right">1mil = 0.0254mm</text>
-<text x="304.508" y="31.238" size="1.27" layer="22" font="vector" rot="MR0">1mil = 1/1000 in</text>
+<text x="303.7" y="16.8" size="1.778" layer="21" font="vector" ratio="15" align="bottom-right">1mm = 39.3701mil</text>
+<text x="303.7" y="14.2" size="1.778" layer="21" font="vector" ratio="15" align="bottom-right">1mil = 0.0254mm</text>
+<text x="304.508" y="31.238" size="1.27" layer="22" font="vector" ratio="15" rot="MR0">1mil = 1/1000 in</text>
 <rectangle x1="299.212" y1="28.956" x2="304.8" y2="29.083" layer="22"/>
+<text x="278.13" y="1.27" size="1.778" layer="1" font="vector" ratio="15">V01</text>
+<text x="145.796" y="-9.144" size="1.778" layer="51" font="vector" ratio="15">Michelle Shorter</text>
 </plain>
 <attributes>
@@
 <element name="E$2" library="SparkFun-Hardware" package="STAND-OFF" value="" x="302.26" y="2.54" rot="MR0"/>
 <element name="E$3" library="SparkFun-Hardware" package="STAND-OFF" value="" x="2.54" y="2.54" rot="MR0"/>
-<element name="FRAME1" library="SparkFun-Aesthetics" package="CREATIVE_COMMONS" value="FRAME-LETTER" x="281.94" y="-10.16" rot="MR0"/>
+<element name="FRAME1" library="SparkFun-Aesthetics" package="CREATIVE_COMMONS" value="FRAME-LETTER" x="114.3" y="-8.89"/>
 <element name="LOGO1" library="SparkFun-Aesthetics" package="OSHW-LOGO-M" value="OSHW-LOGOM" x="152.4" y="20.32" rot="MR0"/>
 <element name="U$1" library="BJT_NPN#png" package="BJT_NPN#PNG" value="" x="204.47" y="16.51" rot="MR0"/>
@@
 <element name="U$7" library="Zener#png" package="ZENER#PNG" value="" x="139.7" y="24.13" rot="MR0"/>
 <element name="U$8" library="morse#png" package="MORSE#PNG" value="" x="257.81" y="19.05" rot="MR0"/>
+<element name="U$9" library="SparkFun-Aesthetics" package="SFE_LOGO_NAME_.2" value="" x="191.77" y="29.21" rot="MR0"/>
+<element name="U$10" library="SparkFun-Aesthetics" package="SFE_LOGO_FLAME_.2" value="" x="207.01" y="29.21" rot="MR0"/>
+<element name="U$11" library="SparkFun-Aesthetics" package="SFE_LOGO_FLAME_.2" value="" x="176.53" y="29.21" rot="MR0"/>
 </elements>
 <signals>

Commit message: For Reds
Updated Morse code and protractor to higher resolution images, moved numbers so they were not hitting copper, moved temperature, moved logos, resized inches markings...
Parts:
- removed U$10: (no value), SparkFun-Aesthetics:SFE_LOGO_FLAME_.2
- removed U$8: (no value), morse#png:MORSE#PNG
- added U$12: (no value), Protractor#jpg:PROTRACTOR#JPG
- added U$13: (no value), MorseHD:MORSE#PNG
- moved U$11 125.7 mm to (301.0, 11.4)
- moved LOGO1 5.08 mm to (152.4, 15.2)
Other:
- board text added: "All holes non-plated"
- board text added: "Color Wavelength Infrared: >760nm Red: 610 - 760nm Orange: 590 - 610nm Yellow: 570 - 590nm Green: 500 - 570nm Blue: 450 - 500nm Violet: 400 - 450nm Ultraviolet: <400nm"
- board text added: "R(series)=R1+R2+...Rn R(parallel)= 1/(1/R1+1/R2+...1/Rn)"
- board text removed: "Color Wavelength Infrared: > 760nm Red: 610 - 760nm Orange: 590 - 610nm Yellow: 570 - 590nm Green: 500 - 570nm Blue: 450 - 500nm Violet: 400 - 450nm Ultraviolet: <400nm"
- board text removed: "R(series)=R1+R2+...Rn R(parallell)= 1/(1/R1+1/R2+...1/Rn)"
